File: boards/ereader_0.1/ereader_0.1.kicad_pcb (KiCad board)
At the start: 4 copper layers, 158.5 x 30 mm, 69 parts, among them J1 USB_C_Receptacle_USB2.0_16P, J2 BATT, J3 Conn_ARM_JTAG_SWD_10, J4 Micro_SD_Card_Det2, P1 FPC24, P2 FPC24, Q1 Si1308EDL, Q2 Si1308EDL, U1 BMD-340-A-R, U2 nPM1300-QEAA-R7, U3 USBLC6-2SC6, U4 IQS323-DFN-12N

Commit message: changes
Connections:
- U2 pad 32: unconnected-(U2-VOUT2-Pad32) -> VSYS
- U2 pad 6: unconnected-(U2-PVSS2-Pad6) -> GND
- U4 pad 13: (no net) -> GND
Routing:
- net GND: track 83.0 -> 86.8 mm, vias 57 -> 59
- net VSYS: track 13.2 -> 15.2 mm, vias 5 -> 6

Commit message: finished bom
Parts:
- C1, C24, C25, C7: value 1uf/25V -> 1u/25v
- C10, C19, C2: value 1u/10v -> 1u/25v
- C11: value 2u2/16v -> 2u2/10v
- C30, C32: value 0.1n/10v -> 0n1/10v
- C34, C35: value 1u/10V -> 1u/25v
- R2, R5: value 0.47r -> 0R47
Changed lines of the file:
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@@
 			)
 		)
-		(property "Value" "1u/10v"
+		(property "Value" "1u/25v"
 			(at 0 1.16 90)
 			(layer "F.Fab")
@@
 			)
 		)
-		(property "Value" "0.1n/10v"
+		(property "Value" "0n1/10v"
 			(at 0 1.16 0)
 			(layer "F.Fab")
@@
 			)
 		)
-		(property "Value" "1u/10V"
+		(property "Value" "1u/25v"
 			(at 0 1.16 90)
 			(layer "F.Fab")
@@
 			)
 		)
-		(property "Value" "1uf/25V"
+		(property "Value" "1u/25v"
 			(at 0 1.16 90)
 			(layer "F.Fab")
@@
 			)
 		)
-		(property "Value" "1u/10v"
+		(property "Value" "1u/25v"
 			(at 0 1.16 0)
 			(layer "F.Fab")
@@
 			)
 		)
-		(property "Value" "1u/10V"
+		(property "Value" "1u/25v"
 			(at 0 1.16 90)
 			(layer "F.Fab")
@@
 			)
 		)
-		(property "Value" "0.47r"
+		(property "Value" "0R47"
 			(at 0 1.17 90)
 			(layer "F.Fab")
@@
 			)
 		)
-		(property "Value" "1u/10v"
+		(property "Value" "1u/25v"
 			(at 0 1.16 90)
 			(layer "F.Fab")
@@
 			)
 		)
-		(property "Value" "1uf/25V"
+		(property "Value" "1u/25v"
 			(at 0 1.16 90)
 			(layer "F.Fab")
@@
 			)
 		)
-		(property "Value" "2u2/16v"
+		(property "Value" "2u2/10v"
 			(at 0 1.16 0)
 			(layer "F.Fab")
@@
 			)
 		)
-		(property "Value" "0.1n/10v"
+		(property "Value" "0n1/10v"
 			(at 0 1.16 0)
 			(layer "F.Fab")
@@
 			)
 		)
-		(property "Value" "0.47r"
+		(property "Value" "0R47"
 			(at 0 1.17 90)
 			(layer "F.Fab")
@@
 			)
 		)
-		(property "Value" "1uf/25V"
+		(property "Value" "1u/25v"
 			(at 0 1.16 90)
 			(layer "F.Fab")
@@
 			)
 		)
-		(property "Value" "1uf/25V"
+		(property "Value" "1u/25v"
 			(at 0 1.16 90)
 			(layer "F.Fab")
