File: boards/ereader_0.1/power.kicad_sch (KiCad schematic)
At the start: 14 parts, among them J1 USB_C_Receptacle_USB2.0_16P, J2 BATT, U2 nPM1300-QEAA-R7, U3 USBLC6-2SC6

Commit message: changes
Connections:
- net GND: now also U2.6 (PVSS2)
- net VSYS: now also U2.32 (VOUT2)
- no-connect marks 11 -> 9
Changed lines of the file:
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@@
-	)
-	(no_connect
-		(at 173.99 78.74)
 	)
 	(no_connect
@@
 		(at 173.99 93.98)
 	)
-	(no_connect
-		(at 173.99 83.82)
-	)
 	(wire
 		(pts
@@
 	(wire
 		(pts
+			(xy 175.26 78.74) (xy 175.26 77.47)
+		)
+		(stroke
+			(width 0)
+			(type default)
+		)
+	)
+	(wire
+		(pts
 			(xy 123.19 86.36) (xy 128.27 86.36)
 		)
@@
 	(wire
 		(pts
+			(xy 173.99 83.82) (xy 175.26 83.82)
+		)
+		(stroke
+			(width 0)
+			(type default)
+		)
+	)
+	(wire
+		(pts
 			(xy 93.98 45.72) (xy 93.98 46.99)
 		)
@@
 	(wire
 		(pts
+			(xy 175.26 83.82) (xy 175.26 85.09)
+		)
+		(stroke
+			(width 0)
+			(type default)
+		)
+	)
+	(wire
+		(pts
 			(xy 109.22 53.34) (xy 110.49 53.34)
 		)
@@
 		(pts
 			(xy 66.04 43.18) (xy 62.23 43.18)
+		)
+		(stroke
+			(width 0)
+			(type default)
+		)
+	)
+	(wire
+		(pts
+			(xy 173.99 78.74) (xy 175.26 78.74)
 		)
 		(stroke
@@
 				(path "/653bb34e-da0b-4e65-b882-449d139ca154/07f3e117-9b9e-4524-a44c-718345fed38d"
 					(reference "C15")
+					(unit 1)
+				)
+			)
+		)
+	)
+	(symbol
+		(lib_id "power:+3V3")
+		(at 175.26 77.47 0)
+		(unit 1)
+		(body_style 1)
+		(exclude_from_sim no)
+		(in_bom yes)
+		(on_board yes)
+		(in_pos_files yes)
+		(dnp no)
+		(property "Reference" "#PWR065"
+			(at 175.26 81.28 0)
+			(hide yes)
+			(show_name no)
+			(do_not_autoplace no)
+			(effects
+				(font
+					(size 1.27 1.27)
+				)
+			)
+		)
+		(property "Value" "VSYS"
+			(at 175.26 73.66 0)
+			(show_name no)
+			(do_not_autoplace no)
+			(effects
+				(font
+					(size 1.27 1.27)
+				)
+			)
+		)
+		(property "Footprint" ""
+			(at 175.26 77.47 0)
+			(hide yes)
+			(show_name no)
+			(do_not_autoplace no)
+			(effects
+				(font
+					(size 1.27 1.27)
+				)
+			)
+		)
+		(property "Datasheet" ""
+			(at 175.26 77.47 0)
+			(hide yes)
+			(show_name no)
+			(do_not_autoplace no)
+			(effects
+				(font
+					(size 1.27 1.27)
+				)
+			)
+		)
+		(property "Description" "Power symbol creates a global label with name \"+3V3\""
+			(at 175.26 77.47 0)
+			(hide yes)
+			(show_name no)
+			(do_not_autoplace no)
+			(effects
+				(font
+					(size 1.27 1.27)
+				)
+			)
+		)
+		(pin "1"
+		)
+		(instances
+			(project "ereader_0.1"
+				(path "/653bb34e-da0b-4e65-b882-449d139ca154/07f3e117-9b9e-4524-a44c-718345fed38d"
+					(reference "#PWR065")
 					(unit 1)
 				)
@@
 					(unit 1)
 				)
+			)
+		)
+	)
+	(symbol
+		(lib_id "power:GND")
+		(at 175.26 85.09 0)
+		(unit 1)
+		(body_style 1)
+		(exclude_from_sim no)
+		(in_bom yes)
+		(on_board yes)
+		(in_pos_files yes)
+		(dnp no)
+		(fields_autoplaced yes)
+		(property "Reference" "#PWR064"
+			(at 175.26 91.44 0)
+			(hide yes)
+			(show_name no)
+			(do_not_autoplace no)
+			(effects
+				(font
+					(size 1.27 1.27)
+				)
+			)
+		)
+		(property "Value" "GND"
+			(at 175.26 90.17 0)
+			(hide yes)
+			(show_name no)
+			(do_not_autoplace no)
+			(effects
+				(font
+					(size 1.27 1.27)
+				)
+			)
+		)
+		(property "Footprint" ""
+			(at 175.26 85.09 0)
+			(hide yes)
+			(show_name no)
+			(do_not_autoplace no)
+			(effects
+				(font
+					(size 1.27 1.27)
+				)
+			)
+		)
+		(property "Datasheet" ""
+			(at 175.26 85.09 0)
+			(hide yes)
+			(show_name no)
+			(do_not_autoplace no)
+			(effects
+				(font
+					(size 1.27 1.27)
+				)
+			)
+		)
+		(property "Description" "Power symbol creates a global label with name \"GND\" , ground"
+			(at 175.26 85.09 0)
+			(hide yes)
+			(show_name no)
+			(do_not_autoplace no)
+			(effects
+				(font
+					(size 1.27 1.27)
+				)
+			)
+		)
+		(pin "1"
+		)
+		(instances
+			(project "ereader_0.1"
+				(path "/653bb34e-da0b-4e65-b882-449d139ca154/07f3e117-9b9e-4524-a44c-718345fed38d"
+					(reference "#PWR064")
+					(unit 1)
+				)

Commit message: finished bom
Parts:
- C10: value 1u/10v -> 1u/25v
- C11: value 2u2/16v -> 2u2/10v
Changed lines of the file:
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@@
 			)
 		)
-		(property "Value" "2u2/16v"
+		(property "Value" "2u2/10v"
 			(at 119.38 55.88 0)
 			(show_name no)
@@
 			)
 		)
-		(property "Value" "1u/10v"
+		(property "Value" "1u/25v"
 			(at 97.79 43.1799 0)
 			(show_name no)
